File: kicad/k1-aioc/k1-aioc.kicad_sch (KiCad schematic)
At the start: 46 parts, among them J1 12401832E402A, J2 Conn_01x07_Male, Q1 BC847BS, U1 MIC5330-SSYML, U2 STM32F373CBTx, Y1 8MHz/20pF

Commit message: Changed designator of Type C Jack in Schematic
Parts:
- removed C3: 100n, Capacitor_SMD:C_0603_1608Metric, symbol Device:C
- removed U1: MIC5330-SSYML, AIOC:Micrel_MLF-8-1EP_2x2mm_P0.5mm_EP0.6x1.2mm, symbol aioc:MIC5330-SSYML
- added U1: VRD3333, DH2LM-FP:LLP-6 (2x1.8), symbol DH2LM-Sym:VRD3333
- J1: value 12401832E402A -> GT-USB-7010ASV; footprint AIOC:USB_C_Receptacle_Amphenol_12401832E40-2A -> Connector_USB:USB_C_Receptacle_G-Switch_GT-USB-7010ASV
Connections:
- net +3V3: now also U1.5 (VOUT1)
- net GND: now also U1.0 (GND), U1.4 (GND)
- net VIN: now also U1.1 (EN2), U1.2 (VIN), U1.3 (EN1)
- net at C5.1, FB1.2: now also U1.6 (VOUT2)
