File: kicad/k1-aioc/k1-aioc.kicad_pcb (KiCad board)
At the start: 2 copper layers, 21 x 31.5 mm, 47 parts, among them J1 12401832E402A, J2 Conn_01x07_Male, Q1 BC847BS, U1 MIC5330-SSYML, U2 STM32F373CBTx, Y1 8MHz/20pF

Commit message: Made PCB a little bit more affordable
Changed USB C Jack from Amphenol 12401832E402A to G-Switch GT-USB-7010ASV
Changed LDO from MIC5330-SSYML-TR to VRD3333PLX
Parts:
- J1: footprint AIOC:USB_C_Receptacle_Amphenol_12401832E40-2A -> Connector_USB:USB_C_Receptacle_G-Switch_GT-USB-7010ASV
- U1: value MIC5330-SSYML -> VRD3333; footprint AIOC:Micrel_MLF-8-1EP_2x2mm_P0.5mm_EP0.6x1.2mm -> DH2LM-FP:LLP-6 (2x1.8)
- moved U1 1.58 mm to (105.0, 96.3), turned to 0 degrees
- moved J1 0.78 mm to (111.9, 84.3)
Connections:
- C5 pad 1: Net-(C5-Pad1) -> Net-(U1-VOUT2)
- FB1 pad 2: Net-(C5-Pad1) -> Net-(U1-VOUT2)
- U1 pad 2: GND -> /VIN
- U1 pad 3: Net-(C3-Pad1) -> /VIN
- U1 pad 4: /VIN -> GND
- U1 pad 5: /VIN -> +3V3
- U1 pad 6: (no net) -> Net-(U1-VOUT2)
Routing:
- net Net-(U1-VOUT2): track 0.00 -> 5.30 mm
- net /SWO: track 18.1 -> 13.6 mm
- net GND: track 9.36 -> 5.69 mm, vias 62 -> 63
- net Net-(J1-CC1): track 10.1 -> 6.89 mm, vias 2 -> 0
- net Net-(C5-Pad1): track 3.11 -> 0.00 mm
- net +3V3: track 51.0 -> 53.6 mm, vias 5 -> 7
- net Net-(C3-Pad1): track 1.71 -> 0.00 mm
- net /VBUS: track 11.7 -> 10.3 mm
- net /USB-DP: track 13.1 -> 14.4 mm, vias 3 -> 2
- net /VIN: track 11.5 -> 10.6 mm
- net Net-(J1-CC2): track 8.97 -> 9.73 mm
- net /USB-DN: track 14.0 -> 13.9 mm, vias 3 -> 2

Commit message: Corrected silkscreen on bottom
Other:
- board text added: "Improved by DH2LM @ OV S48"
Changed lines of the file:
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@@
 		(tags "USB C Type-C Receptacle SMD")
 		(property "Reference" "J1"
-			(at 0 -5.5 360)
+			(at 0 -5.5 0)
 			(layer "F.SilkS")
 			(effects
@@
 		)
 		(property "Value" "12401832E402A"
-			(at 0 5 360)
+			(at 0 5 0)
 			(layer "F.Fab")
 			(effects
@@
 		)
 		(fp_text user "${REFERENCE}"
-			(at 0 0 360)
+			(at 0 0 0)
 			(layer "F.Fab")
 			(effects
@@
 		)
 	)
+	(gr_text "Improved by\nDH2LM @ OV S48"
+		(at 113.914 102.61 0)
+		(layer "B.SilkS")
+		(effects
+			(font
+				(size 1 1)
+				(thickness 0.2)
+			)
+			(justify mirror)
+		)
+	)
 	(gr_text "BLD"
 		(at 104 88.75 270)
@@
 	)
 	(gr_text "AIOC V1.0"
-		(at 111.5 81.25 0)
+		(at 111.882 82.798 0)
 		(layer "B.SilkS")
 		(effects
@@
 	)
 	(gr_text "S. Kueppers"
-		(at 111.5 82.75 0)
+		(at 111.5 81.02 0)
 		(layer "B.SilkS")
 		(effects

Commit message: Changed designator of Type C Jack in Schematic
Parts:
- J1: value 12401832E402A -> GT-USB-7010ASV
Changed lines of the file:
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@@
 			)
 		)
-		(property "Value" "12401832E402A"
+		(property "Value" "GT-USB-7010ASV"
 			(at 0 5 0)
 			(layer "F.Fab")

Commit message: Corrected LDO
Parts:
- removed C3: 100n, Capacitor_SMD:C_0603_1608Metric
- moved U1 2.84 mm to (105.5, 93.5), turned to 180 degrees
Routing:
- net /VIN: track 10.6 -> 4.02 mm
- net Net-(U1-VOUT2): track 5.30 -> 3.60 mm
- net +3V3: track 53.6 -> 52.8 mm, vias 7 -> 6
- net GND: track 5.69 -> 6.03 mm, vias 63 -> 64
