File: kicad/k1-aioc-cr/k1-aioc.kicad_pcb (KiCad board)
At the start: 2 copper layers, 21 x 31.5 mm, 49 parts, among them J1 GT-USB-7010ASV, J2 Conn_01x07_Male, Q1 MMBT3904, Q2 MMBT3904, U1 XC6206PxxxMR, U2 STM32F373CBTx, U3 XC6206PxxxMR, Y1 8MHz/20pF

Commit message: Made DRC happy regarding errors
Parts:
- J1: value GT-USB-7010ASV -> TYPE-C-31-M-12; footprint Connector_USB:USB_C_Receptacle_G-Switch_GT-USB-7010ASV -> Connector_USB:USB_C_Receptacle_HRO_TYPE-C-31-M-12
- moved C6 0.44 mm to (108.3, 90.1)
Routing:
- net GND: track 11.1 -> 27.4 mm, vias 73 -> 76
- net /VBUS: track 8.46 -> 7.65 mm
- net /VIN: track 10.5 -> 9.75 mm
Other:
- board text added: "AIOC V1i"
- board text removed: "AIOC V1.0"
