File: kicad/k1-aioc-cr/k1-aioc.kicad_sch (KiCad schematic)
At the start: 45 parts, among them J1 GT-USB-7010ASV, J2 Conn_01x07_Male, Q1 BC847BS, U1 VRD3333, U2 STM32F373CBTx, Y1 8MHz/20pF

Commit message: Added Cost reduced version
Parts:
- removed Q1: BC847BS, Package_TO_SOT_SMD:SOT-363_SC-70-6, symbol Device:Q_Dual_NPN_NPN_E1B1C2E2B2C1
- removed U1: VRD3333, DH2LM-FP:LLP-6 (2x1.8), symbol DH2LM-Sym:VRD3333
- added C3: 1u/10V/X5R, Capacitor_SMD:C_0402_1005Metric, symbol Device:C
- added Q1, Q2: MMBT3904, Package_TO_SOT_SMD:SOT-23, symbol Transistor_BJT:MMBT3904
- added U1, U3: XC6206PxxxMR, Package_TO_SOT_SMD:SOT-23-3, symbol Regulator_Linear:XC6206PxxxMR
- C4, C5, C6: value 4.7u/10V/X5R -> 1u/10V/X5R; footprint Capacitor_SMD:C_0603_1608Metric -> Capacitor_SMD:C_0402_1005Metric
- R1, R10, R11, R12, R13: footprint Resistor_SMD:R_0603_1608Metric -> Resistor_SMD:R_0402_1005Metric
Connections:
- net +3V3: now also U1.2 (VO)
- net GND: now also C3.2, Q1.2 (E), Q2.2 (E), U1.1 (GND), U3.1 (GND)
- net VIN: now also C3.1, U1.3 (VI), U3.3 (VI)
- net at C5.1, FB1.2: now also U3.2 (VO)
- net at R13.2: now also Q2.3 (C)
- net at R11.2: now also Q2.1 (B)
- net at R12.2: now also Q1.3 (C)
- net at R10.2: now also Q1.1 (B)
Other:
- moved on the sheet: C6

Commit message: Made DRC happy regarding errors
Parts:
- J1: value GT-USB-7010ASV -> TYPE-C-31-M-12; footprint Connector_USB:USB_C_Receptacle_G-Switch_GT-USB-7010ASV -> Connector_USB:USB_C_Receptacle_HRO_TYPE-C-31-M-12
Changed lines of the file:
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@@
 			)
 		)
-		(property "Value" "GT-USB-7010ASV"
+		(property "Value" "TYPE-C-31-M-12"
 			(at 36.83 27.94 0)
 			(effects
@@
 			)
 		)
-		(property "Footprint" "Connector_USB:USB_C_Receptacle_G-Switch_GT-USB-7010ASV"
+		(property "Footprint" "Connector_USB:USB_C_Receptacle_HRO_TYPE-C-31-M-12"
 			(at 40.64 48.26 0)
 			(effects
